File: card_reader_pcb/eps32-/eps32-.kicad_sch (KiCad schematic)
At the start: 7 parts, among them J1 Screw_Terminal_01x02, U1 PPSM82916VCER, U2 ESP32-WROOM-32E

Commit message: Add files via upload
Parts:
- removed D1: D_Schottky, symbol Device:D_Schottky
- added C1, C2: 10u, symbol Device:C
- added C3: 132u, symbol Device:C
- added C4: 22u, symbol Device:C
- added C5: 0.1u, symbol Device:C
- added C6: 470n, symbol Device:C
- added FB1: FerriteBead, symbol Device:FerriteBead
- added J2: Conn_01x08, symbol Connector_Generic:Conn_01x08
- added R1: 15.2k, symbol Device:R
- added R2: 4.87k, symbol Device:R
- added R3, R4, R5: R, symbol Device:R
Connections:
- net GND: now also U1.1 (GND), U1.10 (S-conf), U1.13 (GND), U1.15 (GND), U1.4 (PSNS), C2.2, C3.2, C4.2, C6.2, R2.2
- net +12V: now reaches J1.2 (Pin_2)
- net +12V: now also U1.11 (En), U1.12 (Vin), U1.16 (Vin), U1.2 (Vin), C1.1
- net at U1.14 (SW): now also C5.2
- net at U1.3 (Boot): now also C5.1
- net at U1.5 (NR): now also C6.1
- net at U1.6 (FB): now also R1.2, R2.1
- net at U1.7 (Vout): now also U1.8 (VO), C3.1, FB1.2
- new net: C4.1, FB1.1, R1.1
- new net: C1.2, C2.1
- no-connect marks 0 -> 1
Other:
- moved on the sheet: D2, D3, D4, J1, U1, U2

Commit message: Add files via upload
Parts:
- added C10, C7, C8, C9: 22u, symbol Device:C
- added D1: D_Schottky, symbol Device:D_Schottky
- C3: value 132u -> 22u
- C5: value 0.1u -> 22u
Connections:
- net +12V: now also C2.1, D1.1 (K); no longer J1.2 (Pin_2)
- net GND: now also C1.2, C5.2, U1.9 (PG), U2.1 (GND), U2.15 (GND), U2.38 (GND), U2.39 (GND), C10.2, C7.2, C8.2, C9.2
- net +3.3V: now reaches C4.1, FB1.1, R1.1
- net +3.3V: now also U2.2 (VDD)
- net at C3.1, FB1.2, U1.7 (Vout)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: now also C5.1, C10.1, C7.1, C8.1, C9.1
- net at U1.3 (Boot): no longer C5.1
- net at U1.14 (SW): no longer C5.2
- new net: D1.2 (A), J1.2 (Pin_2)
- no-connect marks 1 -> 2
Other:
- moved on the sheet: C1, C2, C3, C4, FB1, J1, J2, R1, R2

Commit message: Add files via upload
Parts:
- added C11: 1u, symbol Device:C
- added R6, R7: 10k, symbol Device:R
- R3: value R -> 50
- R4, R5: value R -> 100
Connections:
- net +3.3V: now also J2.1 (Pin_1), R6.1, R7.2
- net GND: now also D2.1 (K), D3.1 (K), D4.1 (K), J2.3 (Pin_3), U2.4 (SENSOR_VP), U2.5 (SENSOR_VN), C11.2; no longer U1.9 (PG)
- net at D4.2 (A): now also R5.2
- net at D2.2 (A): now also R3.2
- net at D3.2 (A): now also R4.2
- net green: now reaches R3.1
- net green: now also U2.11 (IO26)
- net red: now reaches R5.1
- net red: now also U2.8 (IO32)
- net to_RST: now reaches J2.2 (Pin_2)
- net to_RST: now also U2.36 (IO22)
- net to_MISO: now reaches J2.4 (Pin_4)
- net to_MISO: now also U2.31 (IO19)
- net to_MOSI: now reaches J2.5 (Pin_5)
- net to_MOSI: now also U2.37 (IO23)
- net to_SCK: now reaches J2.6 (Pin_6)
- net to_SCK: now also U2.30 (IO18)
- net to_NSS: now reaches J2.7 (Pin_7)
- net to_NSS: now also U2.29 (IO5)
- net yellow: now reaches R4.1
- net yellow: now also U2.12 (IO27)
- net EN: now reaches U2.3 (EN)
- net EN: now also C11.1, R6.2
- new net PG: R7.1, U1.9 (PG)
- no-connect marks 2 -> 19
Other:
- moved on the sheet: D2, D3, D4, J2, R3, R4, R5, U2

Commit message: Add files via upload
Parts:
- C1, C2: footprint (none) -> Capacitor_SMD:CP_Elec_5x3
- C10, C3, C4, C5, C7, C8, C9: footprint (none) -> Capacitor_SMD:CP_Elec_4x5.3
- C11: footprint (none) -> Capacitor_SMD:CP_Elec_4x5.4
- C6: footprint (none) -> Capacitor_SMD:CP_Elec_4x3
- D1: footprint (none) -> Diode_SMD:D_SMA
- D2, D3, D4: footprint (none) -> LED_SMD:LED_0201_0603Metric
- FB1: footprint (none) -> Ferrite_THT:LairdTech_28C0236-0JW-10
- J1: footprint (none) -> TerminalBlock:TerminalBlock_MaiXu_MX126-5.0-02P_1x02_P5.00mm
- J2: footprint (none) -> Connector_PinSocket_1.00mm:PinSocket_1x08_P1.00mm_Vertical
- R1, R2, R3, R4, R5, R6, R7: footprint (none) -> Resistor_SMD:R_0603_1608Metric
- U1: footprint VCE0016A-MFG -> PPSM82916VCER:VCE0016A-MFG
- U2: footprint RF_Module:ESP32-WROOM-32D -> RF_Module:ESP32-WROOM-32E
Connections:
- net to_RST: now also U2.10 (IO25); no longer U2.36 (IO22)
Changed lines of the file:
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@@
 	)
 	(no_connect
+		(at 96.52 144.78)
+	)
+	(no_connect
 		(at 96.52 165.1)
 	)
@@
 	)
 	(no_connect
-		(at 96.52 149.86)
-	)
-	(no_connect
 		(at 96.52 106.68)
 	)
@@
 	(wire
 		(pts
-			(xy 96.52 144.78) (xy 100.33 144.78)
-		)
-		(stroke
-			(width 0)
-			(type default)
-		)
-	)
-	(wire
-		(pts
 			(xy 195.58 41.91) (xy 203.2 41.91)
 		)
@@
 	(wire
 		(pts
+			(xy 96.52 149.86) (xy 100.33 149.86)
+		)
+		(stroke
+			(width 0)
+			(type default)
+		)
+	)
+	(wire
+		(pts
 			(xy 132.08 62.23) (xy 133.35 62.23)
 		)
@@
 	)
 	(label "to_RST"
-		(at 100.33 144.78 0)
+		(at 100.33 149.86 0)
 		(effects
 			(font
@@
 			)
 		)
-		(property "Footprint" ""
+		(property "Footprint" "Capacitor_SMD:CP_Elec_4x5.4"
 			(at 45.4152 135.89 0)
 			(effects
@@
 			)
 		)
-		(property "Footprint" ""
+		(property "Footprint" "LED_SMD:LED_0201_0603Metric"
 			(at 148.59 163.83 0)
 			(effects
@@
 			)
 		)
-		(property "Footprint" ""
+		(property "Footprint" "Ferrite_THT:LairdTech_28C0236-0JW-10"
 			(at 207.01 40.132 90)
 			(effects
@@
 					(size 1.27 1.27)
 				)
-				(hide yes)
 			)
 		)
@@
 			)
 		)
-		(property "Footprint" ""
+		(property "Footprint" "LED_SMD:LED_0201_0603Metric"
 			(at 148.59 140.97 0)
 			(effects
@@
 			)
 		)
-		(property "Footprint" ""
+		(property "Footprint" "LED_SMD:LED_0201_0603Metric"
 			(at 148.59 152.4 0)
 			(effects
@@
 			)
 		)
-		(property "Footprint" ""
+		(property "Footprint" "TerminalBlock:TerminalBlock_MaiXu_MX126-5.0-02P_1x02_P5.00mm"
 			(at 22.86 29.21 0)
 			(effects
@@
 			)
 		)
-		(property "Footprint" ""
+		(property "Footprint" "Capacitor_SMD:CP_Elec_5x3"
 			(at 64.4652 36.83 0)
 			(effects
@@
 			)
 		)
-		(property "Footprint" ""
+		(property "Footprint" "Capacitor_SMD:CP_Elec_4x5.3"
 			(at 155.9052 50.8 0)
 			(effects
@@
 			)
 		)
-		(property "Footprint" ""
+		(property "Footprint" "Resistor_SMD:R_0603_1608Metric"
 			(at 135.89 142.748 90)
 			(effects
@@
 			)
 		)
-		(property "Footprint" ""
+		(property "Footprint" "Diode_SMD:D_SMA"
 			(at 34.29 26.67 0)
 			(effects
@@
 			)
 		)
-		(property "Footprint" ""
+		(property "Footprint" "Capacitor_SMD:CP_Elec_4x5.3"
 			(at 144.4752 50.8 0)
 			(effects
@@
 			)
 		)
-		(property "Footprint" ""
+		(property "Footprint" "Resistor_SMD:R_0603_1608Metric"
 			(at 42.672 119.38 90)
 			(effects
@@
 			)
 		)
-		(property "Footprint" ""
+		(property "Footprint" "Capacitor_SMD:CP_Elec_4x5.3"
 			(at 196.5452 50.8 0)
 			(effects
@@
 			)
 		)
-		(property "Footprint" ""
+		(property "Footprint" "Resistor_SMD:R_0603_1608Metric"
 			(at 135.89 165.608 90)
 			(effects
@@
 			)
 		)
-		(property "Footprint" ""
+		(property "Footprint" "Connector_PinSocket_1.00mm:PinSocket_1x08_P1.00mm_Vertical"
 			(at 151.13 113.03 0)
 			(effects
@@
 					(size 1.27 1.27)
 				)
-				(hide yes)
 			)
 		)
@@
 			)
 		)
-		(property "Footprint" ""
+		(property "Footprint" "Resistor_SMD:R_0603_1608Metric"
 			(at 135.89 154.178 90)
 			(effects
@@
 			)
 		)
-		(property "Footprint" "VCE0016A-MFG"
+		(property "Footprint" "PPSM82916VCER:VCE0016A-MFG"
 			(at 91.44 26.67 0)
 			(effects
@@
 			)
 		)
-		(property "Footprint" ""
+		(property "Footprint" "Capacitor_SMD:CP_Elec_4x5.3"
 			(at 176.2252 50.8 0)
 			(effects
@@
 			)
 		)
-		(property "Footprint" ""
+		(property "Footprint" "Resistor_SMD:R_0603_1608Metric"
 			(at 210.312 53.34 90)
 			(effects
@@
 			)
 		)
-		(property "Footprint" ""
+		(property "Footprint" "Capacitor_SMD:CP_Elec_4x5.3"
 			(at 186.3852 50.8 0)
 			(effects
@@
 			)
 		)
-		(property "Footprint" ""
+		(property "Footprint" "Resistor_SMD:R_0603_1608Metric"
 			(at 210.312 66.04 90)
 			(effects
@@
 			)
 		)
-		(property "Footprint" ""
+		(property "Footprint" "Resistor_SMD:R_0603_1608Metric"
 			(at 162.56 28.448 90)
 			(effects
@@
 			)
 		)
-		(property "Footprint" ""
+		(property "Footprint" "Capacitor_SMD:CP_Elec_4x5.3"
 			(at 228.2952 59.69 0)
 			(effects
@@
 			)
 		)
-		(property "Footprint" ""
+		(property "Footprint" "Capacitor_SMD:CP_Elec_4x5.3"
 			(at 166.0652 50.8 0)
 			(effects
@@
 			)
 		)
-		(property "Footprint" ""
+		(property "Footprint" "Capacitor_SMD:CP_Elec_4x3"
 			(at 87.3252 73.66 0)
 			(effects
@@
 			)
 		)
-		(property "Footprint" ""
+		(property "Footprint" "Capacitor_SMD:CP_Elec_5x3"
 			(at 75.8952 36.83 0)
 			(effects
@@
 			)
 		)
-		(property "Footprint" "RF_Module:ESP32-WROOM-32D"
+		(property "Footprint" "RF_Module:ESP32-WROOM-32E"
 			(at 97.79 171.45 0)
 			(effects

Commit message: Add files via upload
Parts:
- removed C10, C5, C7, C8, C9: 22u, Capacitor_SMD:CP_Elec_4x5.3, symbol Device:C
- removed C6: 470n, Capacitor_SMD:CP_Elec_4x3, symbol Device:C
- removed FB1: FerriteBead, Ferrite_THT:LairdTech_28C0236-0JW-10, symbol Device:FerriteBead
- removed U1: PPSM82916VCER, PPSM82916VCER:VCE0016A-MFG, symbol TPSM82916:PPSM82916VCER
- added BZ1: Buzzer, Buzzer_Beeper:Buzzer_TDK_PS1240P02BT_D12.2mm_H6.5mm, symbol Device:Buzzer
- added C12, C13: 100n, Capacitor_SMD:C_0201_0603Metric, symbol Device:C
- added D5: 75V 300mA, Diode_SMD:D_0201_0603Metric, symbol Device:D
- added J3: Conn_01x05_Socket, Connector_PinHeader_1.00mm:PinHeader_1x05_P1.00mm_Vertical, symbol Connector:Conn_01x05_Socket
- added J4: Screw_Terminal_01x02, TerminalBlock:TerminalBlock_MaiXu_MX126-5.0-02P_1x02_P5.00mm, symbol Connector:Screw_Terminal_01x02
- added K2: Relay_SPST-NO, Relay_THT:Relay_SPST_Finder_32.21-x300, symbol Relay:Relay_SPST-NO
- added L1: 15u, Inductor_SMD:L_6.3x6.3_H3, symbol Device:L
- added Q1: Q_NPN_BCE, Package_TO_SOT_SMD:SOT-23, symbol Transistor_BJT:Q_NPN_BCE
- added R8: 100, Resistor_SMD:R_0603_1608Metric, symbol Device:R
- added R9: 1k, Resistor_SMD:R_0603_1608Metric, symbol Device:R
- added U1: LMR51610XFQDBVRQ1, LMR516:DBV0006A-IPC_C, symbol LMR51610XFQDBVRQ1:LMR51610XFQDBVRQ1
- C1: value 10u -> 3.3u; footprint Capacitor_SMD:CP_Elec_5x3 -> Capacitor_SMD:C_0201_0603Metric
- C11: footprint Capacitor_SMD:CP_Elec_4x5.4 -> Capacitor_SMD:C_0201_0603Metric
- C2: value 10u -> 100n; footprint Capacitor_SMD:CP_Elec_5x3 -> Capacitor_SMD:C_0201_0603Metric
- C3: value 22u -> 100n; footprint Capacitor_SMD:CP_Elec_4x5.3 -> Capacitor_SMD:C_0201_0603Metric
- C4: value 22u -> 10u; footprint Capacitor_SMD:CP_Elec_4x5.3 -> Capacitor_SMD:C_0201_0603Metric
- D1: value D_Schottky -> 40V 3A; footprint Diode_SMD:D_SMA -> Diode_SMD:D_0402_1005Metric
- R1: value 15.2k -> 100k
- R2: value 4.87k -> 32k
- R3: value 50 -> 1k
- R4, R5: value 100 -> 1k
Connections:
- net PG is gone; now on net +3.3V: R7.1
- net +12V: now also D5.1 (K), K2.A2, U1.4 (EN), U1.5 (VIN)
- net +3.3V: now also L1.2; no longer R7.2
- net EN: now also C13.1
- net GND: now also BZ1.2 (-), J3.1 (Pin_1), Q1.3 (E), U1.2 (GND); no longer C3.2
- net at C3.1: now also U1.1 (CB)
- net at R1.2, R2.1: now also U1.3 (FB)
- net BUZZER: now reaches U2.16 (IO13)
- net BUZZER: now also R8.1
- net RELAY: now reaches U2.23 (IO15)
- net RELAY: now also R9.1
- net IO0: now reaches U2.25 (IO0)
- net IO0: now also R7.2, C12.1
- net TXD: now reaches U2.34 (RXD0/IO3)
- net TXD: now also J3.2 (Pin_2)
- net RXD: now reaches U2.35 (TXD0/IO1)
- net RXD: now also J3.3 (Pin_3)
- new net: C3.2, L1.1, U1.6 (SW)
- new net: Q1.1 (B), R9.2
- new net: BZ1.1 (+), R8.2
- new net: D5.2 (A), K2.A1, Q1.2 (C)
- new net: J4.1 (Pin_1), K2.14
- new net: J4.2 (Pin_2), K2.13
- new net BOOT: C12.2, J3.5 (Pin_5)
- new net RST: C13.2, J3.4 (Pin_4)
- no-connect marks 19 -> 12
Other:
- note added: "1A"
- moved on the sheet: C11, D1, D2, D3, D4, J1, J2, R3, R4, R5, R6, U2
